Commit message: 修改了ComputeSkidRate中计算两个link相对位姿的函数ComputeRelativePose()，似乎gazebo官方插件gazebo_ros_p3d中求解两个link相对位姿的代码存在错误，具体见/pluginplugins/ComputeSkidRate/src/ComputeSkidRate.cpp的319行左右。

File: urdf/MarsRover.xacro (robot description, xacro)
@@ -1122,43 +1122,3 @@
   <xacro:PandarQT link="${LidarName}" topic="${LidarDataTopicName}" hz="${LidarHz}" lasers="${LidarLasers}" samples="${LidarSamples}" visual="${LidarBeamVisual}"></xacro:PandarQT>
   <xacro:IMU link="${LidarName}" pitch="${0}" gaussianNoise="0.0"></xacro:IMU>
-<!--   <transmission name="trans_RightMainRocket_BogieRF">
-    <type>transmission_interface/SimpleTransmission</type>
-    <joint name="c_RightMainRocket_BogieRF">
-      <hardwareInterface>hardware_interface/EffortJointInterface</hardwareInterface>
-    </joint>
-    <actuator name="motor1">
-      <hardwareInterface>EffortJointInterface</hardwareInterface>
-      <mechanicalReduction>1</mechanicalReduction>
-    </actuator>
-  </transmission>
-  <transmission name="trans_LeftMainRocket_BogieLF">
-    <type>transmission_interface/SimpleTransmission</type>
-    <joint name="c_LeftMainRocket_BogieLF">
-      <hardwareInterface>hardware_interface/EffortJointInterface</hardwareInterface>
-    </joint>
-    <actuator name="motor2">
-      <hardwareInterface>EffortJointInterface</hardwareInterface>
-      <mechanicalReduction>1</mechanicalReduction>
-    </actuator>
-  </transmission>
-  <transmission name="trans_RightViceRocket_BogieRR">
-    <type>transmission_interface/SimpleTransmission</type>
-    <joint name="c_RightViceRocket_BogieRR">
-      <hardwareInterface>hardware_interface/EffortJointInterface</hardwareInterface>
-    </joint>
-    <actuator name="motor3">
-      <hardwareInterface>EffortJointInterface</hardwareInterface>
-      <mechanicalReduction>1</mechanicalReduction>
-    </actuator>
-  </transmission>
-  <transmission name="trans_LeftViceRocket_BogieLR">
-    <type>transmission_interface/SimpleTransmission</type>
-    <joint name="c_LeftViceRocket_BogieLR">
-      <hardwareInterface>hardware_interface/EffortJointInterface</hardwareInterface>
-    </joint>
-    <actuator name="motor4">
-      <hardwareInterface>EffortJointInterface</hardwareInterface>
-      <mechanicalReduction>1</mechanicalReduction>
-    </actuator>
-  </transmission> -->
 </robot>

Commit message: 将STL格式的模型文件替换为DAE文件，方便使用Blender设置模型的颜色材质等。

File: urdf/MarsRover.xacro (robot description, xacro)
@@ -35,18 +35,18 @@
       <geometry>
         <mesh
-          filename="package://mars_rover_2/meshes/rover/Body.STL" />
-      </geometry>
-      <material
-        name="">
-        <color
-          rgba="0.75294 0.75294 0.75294 1" />
-      </material>
-    </visual>
-    <collision>
-      <origin
-        xyz="0 0 0"
-        rpy="0 0 0" />
-      <geometry>
-        <mesh filename="package://mars_rover_2/meshes/rover/Body.STL" />
+          filename="package://mars_rover_2/meshes/rover/Body.dae" />
+      </geometry>
+      <material
+        name="">
+        <color
+          rgba="0.75294 0.75294 0.75294 1" />
+      </material>
+    </visual>
+    <collision>
+      <origin
+        xyz="0 0 0"
+        rpy="0 0 0" />
+      <geometry>
+        <mesh filename="package://mars_rover_2/meshes/rover/Body.dae" />
       </geometry>
     </collision>
@@ -74,5 +74,5 @@
       <geometry>
         <mesh
-          filename="package://mars_rover_2/meshes/rover/LiDARBodyCon.STL" />
+          filename="package://mars_rover_2/meshes/rover/LiDARBodyCon.dae" />
       </geometry>
       <material
@@ -88,5 +88,5 @@
       <geometry>
         <mesh
-          filename="package://mars_rover_2/meshes/rover/LiDARBodyCon.STL" />
+          filename="package://mars_rover_2/meshes/rover/LiDARBodyCon.dae" />
       </geometry>
     </collision>
@@ -127,5 +127,5 @@
       <geometry>
         <mesh
-          filename="package://mars_rover_2/meshes/rover/LiDARSupport.STL" />
+          filename="package://mars_rover_2/meshes/rover/LiDARSupport.dae" />
       </geometry>
       <material
@@ -141,5 +141,5 @@
       <geometry>
         <mesh
-          filename="package://mars_rover_2/meshes/rover/LiDARSupport.STL" />
+          filename="package://mars_rover_2/meshes/rover/LiDARSupport.dae" />
       </geometry>
     </collision>
@@ -185,5 +185,5 @@
       <geometry>
         <mesh
-          filename="package://mars_rover_2/meshes/rover/LiDAR.STL" />
+          filename="package://mars_rover_2/meshes/rover/LiDAR.dae" />
       </geometry>
       <material
@@ -199,5 +199,5 @@
       <geometry>
         <mesh
-          filename="package://mars_rover_2/meshes/rover/LiDAR.STL" />
+          filename="package://mars_rover_2/meshes/rover/LiDAR.dae" />
       </geometry>
     </collision>
@@ -238,19 +238,19 @@
       <geometry>
         <mesh
-          filename="package://mars_rover_2/meshes/rover/DiffBar.STL" />
-      </geometry>
-      <material
-        name="">
-        <color
-          rgba="0.75294 0.75294 0.75294 1" />
-      </material>
-    </visual>
-    <collision>
-      <origin
-        xyz="0 0 0"
-        rpy="0 0 0" />
-      <geometry>
-        <mesh
-          filename="package://mars_rover_2/meshes/rover/DiffBar.STL" />
+          filename="package://mars_rover_2/meshes/rover/DiffBar.dae" />
+      </geometry>
+      <material
+        name="">
+        <color
+          rgba="0.75294 0.75294 0.75294 1" />
+      </material>
+    </visual>
+    <collision>
+      <origin
+        xyz="0 0 0"
+        rpy="0 0 0" />
+      <geometry>
+        <mesh
+          filename="package://mars_rover_2/meshes/rover/DiffBar.dae" />
       </geometry>
     </collision>
@@ -292,19 +292,19 @@
       <geometry>
         <mesh
-          filename="package://mars_rover_2/meshes/rover/RightDiffBarLink.STL" />
-      </geometry>
-      <material
-        name="">
-        <color
-          rgba="0.75294 0.75294 0.75294 1" />
-      </material>
-    </visual>
-    <collision>
-      <origin
-        xyz="0 0 0"
-        rpy="0 0 0" />
-      <geometry>
-        <mesh
-          filename="package://mars_rover_2/meshes/rover/RightDiffBarLink.STL" />
+          filename="package://mars_rover_2/meshes/rover/RightDiffBarLink.dae" />
+      </geometry>
+      <material
+        name="">
+        <color
+          rgba="0.75294 0.75294 0.75294 1" />
+      </material>
+    </visual>
+    <collision>
+      <origin
+        xyz="0 0 0"
+        rpy="0 0 0" />
+      <geometry>
+        <mesh
+          filename="package://mars_rover_2/meshes/rover/RightDiffBarLink.dae" />
       </geometry>
     </collision>
@@ -345,19 +345,19 @@
       <geometry>
         <mesh
-          filename="package://mars_rover_2/meshes/rover/LeftDiffBarLink.STL" />
-      </geometry>
-      <material
-        name="">
-        <color
-          rgba="0.75294 0.75294 0.75294 1" />
-      </material>
-    </visual>
-    <collision>
-      <origin
-        xyz="0 0 0"
-        rpy="0 0 0" />
-      <geometry>
-        <mesh
-          filename="package://mars_rover_2/meshes/rover/LeftDiffBarLink.STL" />
+          filename="package://mars_rover_2/meshes/rover/LeftDiffBarLink.dae" />
+      </geometry>
+      <material
+        name="">
+        <color
+          rgba="0.75294 0.75294 0.75294 1" />
+      </material>
+    </visual>
+    <collision>
+      <origin
+        xyz="0 0 0"
+        rpy="0 0 0" />
+      <geometry>
+        <mesh
+          filename="package://mars_rover_2/meshes/rover/LeftDiffBarLink.dae" />
       </geometry>
     </collision>
@@ -399,19 +399,19 @@
       <geometry>
         <mesh
-          filename="package://mars_rover_2/meshes/rover/RightMainRocket.STL" />
-      </geometry>
-      <material
-        name="">
-        <color
-          rgba="0.75294 0.75294 0.75294 1" />
-      </material>
-    </visual>
-    <collision>
-      <origin
-        xyz="0 0 0"
-        rpy="0 0 0" />
-      <geometry>
-        <mesh
-          filename="package://mars_rover_2/meshes/rover/RightMainRocket.STL" />
+          filename="package://mars_rover_2/meshes/rover/RightMainRocket.dae" />
+      </geometry>
+      <material
+        name="">
+        <color
+          rgba="0.75294 0.75294 0.75294 1" />
+      </material>
+    </visual>
+    <collision>
+      <origin
+        xyz="0 0 0"
+        rpy="0 0 0" />
+      <geometry>
+        <mesh
+          filename="package://mars_rover_2/meshes/rover/RightMainRocket.dae" />
       </geometry>
     </collision>
@@ -452,19 +452,19 @@
       <geometry>
         <mesh
-          filename="package://mars_rover_2/meshes/rover/BogieRF.STL" />
-      </geometry>
-      <material
-        name="">
-        <color
-          rgba="0.75294 0.75294 0.75294 1" />
-      </material>
-    </visual>
-    <collision>
-      <origin
-        xyz="0 0 0"
-        rpy="0 0 0" />
-      <geometry>
-        <mesh
-          filename="package://mars_rover_2/meshes/rover/BogieRF.STL" />
+          filename="package://mars_rover_2/meshes/rover/BogieRF.dae" />
+      </geometry>
+      <material
+        name="">
+        <color
+          rgba="0.75294 0.75294 0.75294 1" />
+      </material>
+    </visual>
+    <collision>
+      <origin
+        xyz="0 0 0"
+        rpy="0 0 0" />
+      <geometry>
+        <mesh
+          filename="package://mars_rover_2/meshes/rover/BogieRF.dae" />
       </geometry>
     </collision>
@@ -505,19 +505,19 @@
       <geometry>
         <mesh
-          filename="package://mars_rover_2/meshes/rover/WheelRF.STL" />
-      </geometry>
-      <material
-        name="">
-        <color
-          rgba="0.75294 0.75294 0.75294 1" />
-      </material>
-    </visual>
-    <collision>
-      <origin
-        xyz="0 0 0"
-        rpy="0 0 0" />
-      <geometry>
-        <mesh
-          filename="package://mars_rover_2/meshes/rover/WheelRF.STL" />
+          filename="package://mars_rover_2/meshes/rover/WheelRF.dae" />
+      </geometry>
+      <material
+        name="">
+        <color
+          rgba="0.75294 0.75294 0.75294 1" />
+      </material>
+    </visual>
+    <collision>
+      <origin
+        xyz="0 0 0"
+        rpy="0 0 0" />
+      <geometry>
+        <mesh
+          filename="package://mars_rover_2/meshes/rover/WheelRF.dae" />
       </geometry>
     </collision>
@@ -558,19 +558,19 @@
       <geometry>
         <mesh
-          filename="package://mars_rover_2/meshes/rover/RightViceRocket.STL" />
-      </geometry>
-      <material
-        name="">
-        <color
-          rgba="0.75294 0.75294 0.75294 1" />
-      </material>
-    </visual>
-    <collision>
-      <origin
-        xyz="0 0 0"
-        rpy="0 0 0" />
-      <geometry>
-        <mesh
-          filename="package://mars_rover_2/meshes/rover/RightViceRocket.STL" />
+          filename="package://mars_rover_2/meshes/rover/RightViceRocket.dae" />
+      </geometry>
+      <material
+        name="">
+        <color
+          rgba="0.75294 0.75294 0.75294 1" />
+      </material>
+    </visual>
+    <collision>
+      <origin
+        xyz="0 0 0"
+        rpy="0 0 0" />
+      <geometry>
+        <mesh
+          filename="package://mars_rover_2/meshes/rover/RightViceRocket.dae" />
       </geometry>
     </collision>
@@ -611,19 +611,19 @@
       <geometry>
         <mesh
-          filename="package://mars_rover_2/meshes/rover/WheelRM.STL" />
-      </geometry>
-      <material
-        name="">
-        <color
-          rgba="0.75294 0.75294 0.75294 1" />
-      </material>
-    </visual>
-    <collision>
-      <origin
-        xyz="0 0 0"
-        rpy="0 0 0" />
-      <geometry>
-        <mesh
-          filename="package://mars_rover_2/meshes/rover/WheelRM.STL" />
+          filename="package://mars_rover_2/meshes/rover/WheelRM.dae" />
+      </geometry>
+      <material
+        name="">
+        <color
+          rgba="0.75294 0.75294 0.75294 1" />
+      </material>
+    </visual>
+    <collision>
+      <origin
+        xyz="0 0 0"
+        rpy="0 0 0" />
+      <geometry>
+        <mesh
+          filename="package://mars_rover_2/meshes/rover/WheelRM.dae" />
       </geometry>
     </collision>
@@ -664,19 +664,19 @@
       <geometry>
         <mesh
-          filename="package://mars_rover_2/meshes/rover/BogieRR.STL" />
-      </geometry>
-      <material
-        name="">
-        <color
-          rgba="0.75294 0.75294 0.75294 1" />
-      </material>
-    </visual>
-    <collision>
-      <origin
-        xyz="0 0 0"
-        rpy="0 0 0" />
-      <geometry>
-        <mesh
-          filename="package://mars_rover_2/meshes/rover/BogieRR.STL" />
+          filename="package://mars_rover_2/meshes/rover/BogieRR.dae" />
+      </geometry>
+      <material
+        name="">
+        <color
+          rgba="0.75294 0.75294 0.75294 1" />
+      </material>
+    </visual>
+    <collision>
+      <origin
+        xyz="0 0 0"
+        rpy="0 0 0" />
+      <geometry>
+        <mesh
+          filename="package://mars_rover_2/meshes/rover/BogieRR.dae" />
       </geometry>
     </collision>
@@ -717,19 +717,19 @@
       <geometry>
         <mesh
-          filename="package://mars_rover_2/meshes/rover/WheelRR.STL" />
-      </geometry>
-      <material
-        name="">
-        <color
-          rgba="0.75294 0.75294 0.75294 1" />
-      </material>
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